Commit message: add lidar

File: model/robot.xacro (robot description, xacro)
@@ -131,3 +131,29 @@
         <xacro:inertia_caster/>
     </link>
+    <!-- LIDAR -->
+    <joint name="lidar_joint" type="fixed">
+        <origin xyz="0 0 ${b+r}" rpy="0 0 0"/>
+        <parent link="body_link"/>
+        <child link="lidar_link"/>
+        <axis xyz="0 1 0" rpy="0 0 0"/>
+    </joint>
+    <link name="lidar_link">
+        <visual>
+            <origin rpy="0 0 0.05" xyz="0 0 0"/>
+            <geometry>
+                <cylinder length="0.1" radius="0.1" />
+            </geometry>
+        </visual>
+        <collision name="collision">
+            <origin rpy="0 0 0.05" xyz="0 0 0"/>
+            <geometry>
+                <cylinder length="0.1" radius="0.1" />
+            </geometry>
+        </collision>
+        <inertial>
+            <mass value="1e-6"/>
+            <origin rpy="0 0 0" xyz="0 0 0"/>
+            <inertia ixx="1e-6" ixy="0.0" ixz="0.0" iyy="1e-6" iyz="0" izz="1e-6"/>
+        </inertial>
+    </link>
 </robot>
